File: K_relay.kicad_pcb (KiCad board)
At the start: 2 copper layers, 43 parts, among them J1 ANT3, J10 Con_IDC, J11 To CTL, J2 ANT1, J3 ANT2, J4 ANT4, J5 TRX From SDR, J6 FROM ATU OUT, J7 TO ATU IN, J8 FROM LPF, J9 To PA input, K1 TRA2 L-12VDC-S-Z, K2 TRA2 L-12VDC-S-Z, K3 TQ2-12V, K4 TRA2 L-12VDC-S-Z, K5 TRA2 L-12VDC-S-Z

Commit message: traces completed, silk need some cleaning
Parts:
- C1, C10, C11, C12, C13, C14, C15, C16, C17, C18, C19, C2, C20, C3, C4, C5, C6, C7, C8, C9, D1, D3, D4, D5, D6, J1, J2, J3, J4, R1, R2: moved to B.Cu
- moved K2 170.4 mm to (226.6, 102.8), turned to -90 degrees
- moved J7 168.5 mm to (260.0, 118.0)
- moved J5 155.8 mm to (263.0, 69.0)
- moved K1 151.2 mm to (194.0, 87.4)
- moved J8 144.1 mm to (238.0, 118.0)
- moved J9 140.2 mm to (247.5, 68.5)
- moved J1 138.4 mm to (169.0, 106.9), turned to 180 degrees
- moved K3 133.9 mm to (247.2, 81.4), turned to -90 degrees
- moved C3 126.7 mm to (250.5, 89.0)
- moved D6 126.0 mm to (251.0, 99.0), turned to -90 degrees
- moved J11 125.1 mm to (232.0, 68.5)
- moved C2 123.4 mm to (247.5, 84.5), turned to -90 degrees
- moved C11 120.0 mm to (247.5, 103.0), turned to 180 degrees
- moved C10 119.1 mm to (247.5, 95.5), turned to 180 degrees
- moved C1 117.1 mm to (238.5, 92.0), turned to 180 degrees
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Connections:
- J2 pad 1: Net-(J1-In) -> Net-(J2-In)
- J4 pad 1: Net-(J3-In) -> Net-(J4-In)
- K4 pad 2: Net-(J1-In) -> Net-(J2-In)
- K4 pad 7: Net-(J1-In) -> Net-(J2-In)
- K5 pad 4: Net-(J3-In) -> Net-(J4-In)
- K5 pad 5: Net-(J3-In) -> Net-(J4-In)
Routing:
- net +12V: track 0.00 -> 291.0 mm, vias 0 -> 5
- net K5-4: track 0.00 -> 174.9 mm, vias 0 -> 3
- net K2: track 0.00 -> 92.3 mm, vias 0 -> 2
- net K1: track 0.00 -> 69.4 mm
- net K3: track 0.00 -> 62.3 mm, vias 0 -> 4
- net Net-(J7-In): track 0.00 -> 44.1 mm
- net Net-(J5-In): track 0.00 -> 39.7 mm
- net Net-(J6-In): track 0.00 -> 36.8 mm
- net Net-(J1-In): track 0.00 -> 32.9 mm
- net Net-(J8-In): track 0.00 -> 32.5 mm
- net Net-(K1-Pad4): track 0.00 -> 32.3 mm
- net Net-(J4-In): track 0.00 -> 30.8 mm
- net GND: track 0.00 -> 30.7 mm, vias 0 -> 143
- net Net-(J9-In): track 0.00 -> 30.2 mm
- net Net-(K1-Pad2): track 0.00 -> 29.5 mm
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- added copper zone on B.Cu, net GND
- added copper zone on F.Cu, net GND
Other:
- board outline added: 116 x 82 mm
- board text added: "ANT 1"
- board text added: "ANT 2"
- board text added: "ANT 3"
- board text added: "ANT 4"
- board text added: "Ctrl"
- board text added: "From ATU Out"
- board text added: "From LPF"
- board text added: "From TRX"
- board text added: "LA2NI OpenHPSDR Antenna Relay Board"
- board text added: "To ATU In"
- board text added: "To PA In"
- board text added: "to J3 K_Protec board"

Commit message: minor mods in routing, silk cleaned, ibom and gerber ok
Parts:
- added G***: LOGO, Munin-master:Munin, F.Cu at (259.8, 59.6)
- moved J5 8.05 mm to (259.5, 76.2)
Routing:
- net +12V: track 291.0 -> 319.3 mm, vias 5 -> 3
- net K2: track 92.3 -> 112.7 mm, vias 2 -> 0
- net K3: track 62.3 -> 82.1 mm
- net Net-(K1-Pad4): track 32.3 -> 39.5 mm
- net Net-(J5-In): track 39.7 -> 33.2 mm
- net Net-(J6-In): track 36.8 -> 34.8 mm
- net GND: vias 143 -> 130
